File: designs/Sora-Thin-Client-Satu-Layer/Sora-Thin-Client-Satu-Layer.kicad_pcb (KiCad board)
At the start: 2 copper layers, 75.5 x 54.8 mm, 17 parts, among them J1 AudioJackI2C_Switch, Q1 IRLZ44N, SW1 SW_Push, U1 ESP32_DevKit_V1_DOIT

Commit message: fix: lampu wajib horizontal
Parts:
- moved D2 1.59 mm to (162.6, 119.2), turned to 90 degrees
- moved D3 0.92 mm to (156.8, 119.3), turned to 90 degrees
- moved D1 0.71 mm to (157.5, 79.2), turned to 90 degrees
Routing:
- net GND1: track 108.5 -> 120.0 mm
- net Net-(D1-A): track 3.69 -> 4.78 mm

Commit message: fix: memperlebar ukuran supaya mudah pada saat solder
bersama coach sam dkk
Parts:
- D1, D2, D3, D4, SW1: footprint Connector_PinHeader_1.27mm:PinHeader_1x02_P1.27mm_Vertical -> Connector_PinHeader_2.54mm:PinHeader_1x02_P2.54mm_Vertical
- J1: footprint Connector_PinHeader_1.27mm:PinHeader_1x04_P1.27mm_Vertical -> Connector_PinHeader_2.00mm:PinHeader_1x04_P2.00mm_Vertical
- U2: footprint Connector_PinHeader_1.27mm:PinHeader_1x04_P1.27mm_Vertical -> Connector_PinHeader_2.54mm:PinHeader_1x04_P2.54mm_Vertical
- U3: footprint Connector_PinHeader_1.27mm:PinHeader_1x03_P1.27mm_Vertical -> Connector_PinHeader_2.54mm:PinHeader_1x03_P2.54mm_Vertical
- moved U2 4.51 mm to (99.9, 80.5)
- moved SW1 3.49 mm to (99.8, 120.5)
- moved D1 2.10 mm to (159.5, 80.0)
- moved D2 1.92 mm to (164.5, 119.5)
- moved D4 0.68 mm to (152.5, 80.0)
- moved U3 0.50 mm to (143.2, 80.0)
Routing:
- net /PN532_RESET: track 34.1 -> 55.9 mm, vias 0 -> 2
- net /SDA: track 122.0 -> 114.2 mm
- net GND1: track 120.0 -> 115.3 mm, vias 0 -> 2
- net +5V: track 40.6 -> 44.7 mm
- net Net-(Q1-D): track 30.8 -> 34.8 mm
- net Net-(U1-EN): track 39.0 -> 42.4 mm
- net GND2: track 29.6 -> 32.6 mm
- net +3.3V: track 56.3 -> 59.0 mm
- net /SERIAL_SENT_LED: track 29.1 -> 31.6 mm
- net Net-(D1-A): track 4.78 -> 7.00 mm
- net /SCL: track 111.4 -> 109.3 mm
- net /IR_SENSOR: track 36.3 -> 34.5 mm
- net Net-(D2-A): track 7.72 -> 9.28 mm
- net Net-(D3-A): track 8.30 -> 7.77 mm
